File: Acquisition_board_aduino_UNO/Acquisition_board_aduino_UNO.kicad_pcb (KiCad board)
At the start: 2 copper layers, 68.6 x 53.3 mm, 27 parts, among them J1 Conn_01x06_Female, J2 Conn_01x08_Female, J3 Conn_01x04_Female, P1 Power, P2 Analog, P3 Digital, P4 Digital, P5 CONN_01X01, P6 CONN_01X01, P7 CONN_01X01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

Commit message: routing n schematic
Parts:
- added R8: 330, Resistor_THT:R_Axial_DIN0204_L3.6mm_D1.6mm_P2.54mm_Vertical, F.Cu at (151.6, 83.2)
- moved C1 108.8 mm to (136.5, 112.4)
- moved R2 103.7 mm to (134.0, 112.4), turned to 90 degrees
- moved JP1 102.9 mm to (142.7, 98.4), turned to 180 degrees
- moved R3 102.2 mm to (136.5, 109.8)
- moved R5 100.5 mm to (150.7, 109.8), turned to 180 degrees
- moved R4 100.5 mm to (143.1, 109.8)
- moved C3 90.4 mm to (148.2, 114.9)
- moved R1 89.7 mm to (139.3, 98.4), turned to 90 degrees
- moved R6 86.4 mm to (148.2, 112.4)
- moved C2 85.5 mm to (150.4, 106.0)
- moved R7 77.0 mm to (159.6, 95.9), turned to -90 degrees
- moved GS1 73.0 mm to (150.4, 95.9)
- moved D1 56.8 mm to (154.2, 81.9)
- moved Q1 52.0 mm to (173.6, 80.6), turned to -90 degrees
- moved BZ1 42.6 mm to (162.0, 84.5)
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Connections:
- D1 pad 1: GND -> Net-(D1-Pad1)
- P5 pad 1: unconnected-(P5-Pad1) -> GND
- P6 pad 1: unconnected-(P6-Pad1) -> GND
- P7 pad 1: unconnected-(P7-Pad1) -> GND
- P8 pad 1: unconnected-(P8-Pad1) -> GND
Routing:
- net +5V: track 0.00 -> 159.7 mm, vias 0 -> 4
- net GND: track 0.00 -> 65.7 mm, vias 0 -> 12
- net rst_LoRa: track 0.00 -> 56.1 mm
- net Net-(GS1-Pad8): track 0.00 -> 48.9 mm
- net RX_LoRa: track 0.00 -> 43.2 mm
- net RX_BLE: track 0.00 -> 42.3 mm
- net TX_BLE: track 0.00 -> 40.0 mm
- net TX_LoRa: track 0.00 -> 39.7 mm
- net Net-(C2-Pad1): track 0.00 -> 35.5 mm
- net Net-(C2-Pad2): track 0.00 -> 34.4 mm
- net ADC_temp: track 0.00 -> 33.3 mm
- net Display_SDA: track 0.00 -> 26.3 mm
- net ADC_Gas: track 0.00 -> 19.9 mm
- net Display_SCL: track 0.00 -> 17.8 mm
- net Net-(C1-Pad1): track 0.00 -> 13.9 mm
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- added copper zone on F.Cu, net GND
Other:
- board text added: "Mass.Benc.Mich.Caut"
