File: Acquisition_board_aduino_UNO/display.kicad_sch (KiCad schematic)
At the start: 3 parts, among them J3 Conn_01x04_Female

Commit message: routing n schematic
Parts:
- added R8: 330, Resistor_THT:R_Axial_DIN0204_L3.6mm_D1.6mm_P2.54mm_Vertical, symbol Device:R
Connections:
- net GND: now also R8.2; no longer D1.1 (K)
- new net: D1.1 (K), R8.1
Changed lines of the file:
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@@
     (stroke (width 0) (type default) (color 0 0 0 0))
   )
-  (wire (pts (xy 81.28 96.52) (xy 81.28 109.22))
+  (wire (pts (xy 81.28 107.95) (xy 81.28 109.22))
+    (stroke (width 0) (type default) (color 0 0 0 0))
+  )
+  (wire (pts (xy 81.28 96.52) (xy 81.28 100.33))
     (stroke (width 0) (type default) (color 0 0 0 0))
   )
@@
     (pin "4")
   )
+  (symbol (lib_id "Device:R") (at 81.28 104.14 0) (unit 1)
+    (in_bom yes) (on_board yes) (fields_autoplaced)
+    (property "Reference" "R8" (id 0) (at 83.82 102.8699 0)
+      (effects (font (size 1.27 1.27)) (justify left))
+    )
+    (property "Value" "330" (id 1) (at 83.82 105.4099 0)
+      (effects (font (size 1.27 1.27)) (justify left))
+    )
+    (property "Footprint" "Resistor_THT:R_Axial_DIN0204_L3.6mm_D1.6mm_P2.54mm_Vertical" (id 2) (at 79.502 104.14 90)
+      (effects (font (size 1.27 1.27)) hide)
+    )
+    (property "Datasheet" "~" (id 3) (at 81.28 104.14 0)
+      (effects (font (size 1.27 1.27)) hide)
+    )
+    (pin "1")
+    (pin "2")
+  )
   (symbol (lib_id "Device:Buzzer") (at 106.68 91.44 0) (mirror y) (unit 1)
